File: Projects/Charlieplexing/eagle/9x9_backpack.brd (EAGLE design)
At the start: 45.7 x 45.7 mm, 103 parts

Commit message: update contact information
Routing:
- net D: track 190.1 -> 0.00 mm, vias 2 -> 0
- net S8: track 160.4 -> 0.00 mm, vias 2 -> 0
- net S0: track 131.3 -> 0.00 mm, vias 1 -> 0
- net S7: track 129.5 -> 0.00 mm
- net S3: track 123.3 -> 0.00 mm, vias 1 -> 0
- net S6: track 119.2 -> 0.00 mm, vias 1 -> 0
- net S1: track 117.2 -> 0.00 mm, vias 1 -> 0
- net S5: track 115.3 -> 0.00 mm
- net S2: track 107.4 -> 0.00 mm, vias 1 -> 0
- net S4: track 101.0 -> 0.00 mm, vias 3 -> 0
- net S$2: track 84.3 -> 0.00 mm, vias 2 -> 0
- net S$4: track 60.3 -> 0.00 mm, vias 1 -> 0
- net S$3: track 53.4 -> 0.00 mm, vias 4 -> 0
- net S$1: track 40.5 -> 0.00 mm, vias 2 -> 0
- net S$5: track 16.5 -> 0.00 mm, vias 1 -> 0
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Other:
- board text added: "M E Rule"
- board text added: "mrule7404@gmail.com"
- board text removed: "Michael Everett Rule"
- board text removed: "slowdanger@gmail.com"
