File: Projects/Charlieplexing/eagle/old/charlie2/9x9_backpack.brd (EAGLE design)
At the start: 45.7 x 45.7 mm, 103 parts

Commit message: update contact information
Routing:
- net D: track 0.00 -> 190.1 mm, vias 0 -> 2
- net S8: track 0.00 -> 160.4 mm, vias 0 -> 2
- net S0: track 0.00 -> 131.3 mm, vias 0 -> 1
- net S7: track 0.00 -> 129.5 mm
- net S3: track 0.00 -> 123.3 mm, vias 0 -> 1
- net S6: track 0.00 -> 119.2 mm, vias 0 -> 1
- net S1: track 0.00 -> 117.2 mm, vias 0 -> 1
- net S5: track 0.00 -> 115.3 mm
- net S2: track 0.00 -> 107.4 mm, vias 0 -> 1
- net S4: track 0.00 -> 101.0 mm, vias 0 -> 3
- net S$2: track 0.00 -> 84.3 mm, vias 0 -> 2
- net S$4: track 0.00 -> 60.3 mm, vias 0 -> 1
- net S$3: track 0.00 -> 53.4 mm, vias 0 -> 4
- net S$1: track 0.00 -> 40.5 mm, vias 0 -> 2
- net S$5: track 0.00 -> 16.5 mm, vias 0 -> 1
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Other:
- board text added: "M E Rule"
- board text added: "mrule7404@gmail.com"
- board text removed: "Michael Everett Rule"
- board text removed: "slowdanger@gmail.com"
