File: Projects/matrix/eagle/big_8x16.brd (EAGLE design)
At the start: 32 x 64 mm, 39 parts, among them IC1 MEGA8-AI, X1 SSW-104-02-S-S-RA

Commit message: update contact information
Other:
- board text added: "M E Rule"
- board text added: "mrule7404@gmail.com"
- board text removed: "Michael Everett Rule"
- board text removed: "Treehovse Labs"
- board text removed: "slowdanger@gmail.com"
Changed lines of the file:
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@@
 <text x="6" y="23" size="1.016" layer="21" font="vector" ratio="15" rot="R270">.1uF</text>
 <text x="16" y="32" size="1.016" layer="22" font="vector" ratio="15" rot="MR270" align="center">ATMEGA*8</text>
-<text x="26" y="55" size="1.016" layer="22" font="vector" ratio="15" rot="MR90" align="center-right">Michael Everett Rule</text>
-<text x="24" y="55" size="1.016" layer="22" font="vector" ratio="15" rot="MR90" align="center-right">slowdanger@gmail.com</text>
-<text x="22" y="55" size="1.016" layer="22" font="vector" ratio="15" rot="MR270" align="center-left">Treehovse Labs</text>
+<text x="26" y="55" size="1.016" layer="22" font="vector" ratio="15" rot="MR90" align="center-right">M E Rule</text>
+<text x="24" y="55" size="1.016" layer="22" font="vector" ratio="15" rot="MR90" align="center-right">mrule7404@gmail.com</text>
 <text x="10" y="62.875" size="1.016" layer="22" font="vector" ratio="15" rot="MR0" align="center">+</text>
 <text x="22" y="63" size="1.016" layer="22" font="vector" ratio="15" rot="MR0" align="center">-</text>
