File: Projects/matrix/eagle/small_8x16.brd (EAGLE design)
At the start: 20 x 40 mm, 36 parts, among them IC1 MEGA8-AI, X1 SSW-104-02-S-S-RA

Commit message: update contact information
Other:
- board text added: "M E Rule"
- board text added: "mrule7404@gmail.com"
- board text removed: "AS220 Labs"
- board text removed: "Michael Everett Rule"
- board text removed: "Treehovse"
- board text removed: "slowdanger@gmail.com"
Changed lines of the file:
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@@
 <text x="16.5" y="11.75" size="1.016" layer="22" font="vector" ratio="15" rot="MR270">.1uF</text>
 <text x="10" y="20" size="1.016" layer="22" font="vector" ratio="15" rot="MR270" align="center">ATMEGA*8</text>
-<text x="19.25" y="10.5" size="1.016" layer="22" font="vector" ratio="15" rot="MR270" align="center">Michael Everett Rule</text>
-<text x="19.25" y="29.75" size="1.016" layer="22" font="vector" ratio="15" rot="MR270" align="center">slowdanger@gmail.com</text>
-<text x="1" y="33.5" size="1.016" layer="22" font="vector" ratio="15" rot="MR270" align="center">AS220 Labs</text>
-<text x="1" y="6" size="1.016" layer="22" font="vector" ratio="15" rot="MR270" align="center">Treehovse</text>
+<text x="19.25" y="10.5" size="1.016" layer="22" font="vector" ratio="15" rot="MR270" align="center">M E Rule</text>
+<text x="19.25" y="29.75" size="1.016" layer="22" font="vector" ratio="15" rot="MR270" align="center">mrule7404@gmail.com</text>
 <text x="4" y="38.875" size="1.016" layer="22" font="vector" ratio="15" rot="MR0" align="center">+</text>
 <text x="16" y="39" size="1.016" layer="22" font="vector" ratio="15" rot="MR0" align="center">-</text>
