File: Projects/multihex/eagle/9pin_hex.brd (EAGLE design)
At the start: 45.3 x 39.6 mm, 71 parts

Commit message: update contact information
Other:
- board text added: "mrule7404@gmail.com"
- board text removed: "slowdanger@gmail.com"
Changed lines of the file:
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@@
 <text x="22.86" y="34.29" size="1.778" layer="22" font="vector" rot="MR0" align="bottom-center">61566</text>
 <text x="22.225" y="31.115" size="1.778" layer="22" font="vector" rot="MR0" align="center">Michael Everett Rule</text>
-<text x="22.225" y="26.67" size="1.778" layer="22" font="vector" rot="MR0" align="center">slowdanger@gmail.com</text>
+<text x="22.225" y="26.67" size="1.778" layer="22" font="vector" rot="MR0" align="center">mrule7404@gmail.com</text>
 </plain>
 <attributes>
