File: Projects/pov/eagle/tiny13_charlie4_50mm_2xAAA_optical_diag.brd (EAGLE design)
At the start: 100 x 12.5 mm, 22 parts, among them IC1 TINY13-20SSU

Commit message: update contact information
Other:
- board text added: "mrule7404@gmail.com"
- board text removed: "Treehovse"
- board text removed: "slowdanger@gmail.com"
Changed lines of the file:
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@@
 <hole x="99" y="11.5" drill="1"/>
 <hole x="99" y="1" drill="1"/>
-<text x="37.5" y="3.5" size="1.778" layer="21" font="vector">Treehovse</text>
-<text x="37.5" y="1.5" size="1.778" layer="21" font="vector">slowdanger@gmail.com</text>
+<text x="37.5" y="1.5" size="1.778" layer="21" font="vector">mrule7404@gmail.com</text>
 </plain>
 <attributes>
