File: Projects/tetris/eagle/tetris_big_noregulator.brd (EAGLE design)
At the start: 100 x 50 mm, 31 parts, among them IC1 MEGA8-AI, X1 USB-MINIB-5PIN

Commit message: update contact information
Other:
- board text added: "M E Rule"
- board text added: "mrule7404@gmail.com"
- board text removed: "AS220 Labs"
- board text removed: "Michael E. Rule"
- board text removed: "Treehovse"
- board text removed: "slowdanger@gmail.com"
Changed lines of the file:
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@@
 <rectangle x1="71" y1="7" x2="72" y2="8" layer="21"/>
 <rectangle x1="78.5" y1="4" x2="79.5" y2="5" layer="21"/>
-<text x="46" y="41.5" size="1.016" layer="22" font="vector" rot="MR0">Michael E. Rule</text>
-<text x="81" y="41.5" size="1.016" layer="22" font="vector" rot="MR0">slowdanger@gmail.com</text>
-<text x="59.5" y="41.5" size="1.016" layer="22" font="vector" rot="MR0">Treehovse</text>
-<text x="27.5" y="41.5" size="1.016" layer="22" font="vector" rot="MR0">AS220 Labs</text>
+<text x="46" y="41.5" size="1.016" layer="22" font="vector" rot="MR0">M E Rule</text>
+<text x="81" y="41.5" size="1.016" layer="22" font="vector" rot="MR0">mrule7404@gmail.com</text>
 <wire x1="4" y1="9" x2="17" y2="9" width="0.4064" layer="20"/>
 <wire x1="17" y1="9" x2="17" y2="41" width="0.4064" layer="20"/>
