File: Projects/tetris/eagle/tetris_mega_5.brd (EAGLE design)
At the start: 50 x 50 mm, 25 parts, among them IC1 MEGA8-AI, X1 USBPCB

Commit message: update contact information
Other:
- board text added: "M E Rule"
- board text added: "mrule7404@gmail.com"
- board text removed: "Michael Everett Rule"
- board text removed: "slowdanger@gmail.com"
Changed lines of the file:
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@@
 <text x="38.5" y="34" size="0.8128" layer="21" font="vector" ratio="15" rot="R90" align="top-right">Limit</text>
 <text x="32.5" y="34" size="0.8128" layer="21" font="vector" ratio="15" rot="R270">PWR</text>
-<text x="40" y="5" size="0.8128" layer="22" font="vector" ratio="15" rot="MR0" align="center-left">Michael Everett Rule</text>
-<text x="0.5" y="5" size="0.8128" layer="22" font="vector" ratio="15" rot="MR0" align="center-right">slowdanger@gmail.com</text>
+<text x="40" y="5" size="0.8128" layer="22" font="vector" ratio="15" rot="MR0" align="center-left">M E Rule</text>
+<text x="0.5" y="5" size="0.8128" layer="22" font="vector" ratio="15" rot="MR0" align="center-right">mrule7404@gmail.com</text>
 <hole x="20.5" y="31.5" drill="1.2"/>
 <hole x="20.5" y="34.5" drill="1.2"/>
